File: v4220m-eval.kicad_pcb (KiCad board)
At the start: 2 copper layers, 50 x 50 mm, 83 parts, among them J1 POWER, J2 LIN, J3 RIN, J4 IF, J5 LOUT, J6 ROUT, U1 V4220M, U2 NJM8202, U3 NJM8202, U4 NJM8202

Commit message: fix i2s din/dout net
Connections:
- J4 pad 3: /DOUT -> /DIN
- J4 pad 4: /DIN -> /DOUT
- R42 pad 1: /DOUT -> /DIN
- R42 pad 2: /DOUT -> /DIN
- R43 pad 1: /DIN -> /DOUT
- R43 pad 2: /DIN -> /DOUT
- R45 pad 1: /DIN -> /DOUT
- U1 pad 8: /DIN -> /DOUT
- U1 pad 9: /DOUT -> /DIN
